Commit message: several

File: code/resources/pendubot.urdf (robot description, URDF)
Before this commit: robot double_pendulum, 6 links, 5 joints
Joints:
- joint joint1: limit lower=-10000 upper=10000 effort=0.15 velocity=25 -> lower=-10000 upper=10000 effort=0.00 velocity=25
- joint joint2: limit lower=-10000 upper=10000 effort=0.0 velocity=35 -> lower=-10000 upper=10000 effort=0.00 velocity=35

Commit message: velocity cost no reference

File: code/resources/pendubot.urdf (robot description, URDF)
Before this commit: robot double_pendulum, 6 links, 5 joints
Joints:
- joint joint1: limit lower=-10000 upper=10000 effort=0.00 velocity=25 -> lower=-10000 upper=10000 effort=1.5 velocity=25
