Commit message: franka urdf and kkt fix

File: code/resources/urdf/panda/panda.urdf (robot description, URDF)
Before this commit: robot panda, 13 links, 12 joints
Joints:
- joint panda_finger_joint1: axis 0 1 0 -> (none); limit lower=0.0 upper=0.04 effort=20 velocity=0.2 -> (none); type prismatic -> fixed
- joint panda_finger_joint2: axis 0 -1 0 -> (none); limit lower=0.0 upper=0.04 effort=20 velocity=0.2 -> (none); type prismatic -> fixed
